File: hardware/quadcopter.brd (EAGLE design)
At the start: 126.2 x 126.2 mm, 85 parts, among them J1 AVR_SPI_PRG_6-SMD, J2 HEADER-4POS-0.1IN-FEMALE-SMD-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, J3 HEADER-10POSTH-254X10, J4 HEADER-4POS-0.1IN-FEMALE-SMD-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, M1 MOTOR_PADS_GND-MOLEX-SMD, M2 MOTOR_PADS_GND-MOLEX-SMD, M3 MOTOR_PADS_GND-MOLEX-SMD, M4 MOTOR_PADS_GND-MOLEX-SMD, Q1 MOSFET-SI2302CDS-T1-E3CT-ND, Q2 MOSFET-SI2302CDS-T1-E3CT-ND, Q3 MOSFET-SI2302CDS-T1-E3CT-ND, Q4 MOSFET-SI2302CDS-T1-E3CT-ND, Q5 MOSFET-SI2302CDS-T1-E3CT-ND, Q6 MOSFET-SI2302CDS-T1-E3CT-ND, Q7 MOSFET-SI2302CDS-T1-E3CT-ND, Q8 MOSFET-SI2302CDS-T1-E3CT-ND, Q9 MOSFET-SI2302CDS-T1-E3CT-ND, SW1 PUSHBUTTON_SMD-VERTICAL-1, U1 ATMEGA128RFA1, U2 LSM-IMU-497-18367-1-NDIMU, Y1 CRYSTAL5X3

Commit message: fixed full check
Connections:
- net 3V: no longer J1.2
Routing:
- net 3V: track 125.0 -> 101.2 mm, vias 19 -> 16
- net GND: track 66.8 -> 51.2 mm, vias 25 -> 23
Changed lines of the file:
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@@
 <wire x1="11.186" y1="-15.25" x2="17.75" y2="-15.25" width="0.254" layer="16"/>
 <wire x1="17.75" y1="-15.25" x2="21" y2="-12" width="0.254" layer="16"/>
-<via x="10.25" y="12" extent="1-16" drill="0.2032">
-</via>
 <via x="15.5" y="15.75" extent="1-16" drill="0.2032">
 </via>
@@
 <via x="-2" y="0" extent="1-16" drill="0.2032">
 </via>
-<wire x1="10.25" y1="12" x2="11.25" y2="13" width="0.254" layer="1"/>
 <wire x1="11.25" y1="13" x2="11.395" y2="13" width="0.254" layer="1"/>
-<wire x1="22.75" y1="16.855" x2="16.895" y2="11" width="0.254" layer="1"/>
-<wire x1="16.895" y1="11" x2="16.895" y2="10" width="0.254" layer="1"/>
-<wire x1="16.895" y1="10" x2="16.895" y2="8.5" width="0.254" layer="1"/>
-<via x="15" y="8.5" extent="1-16" drill="0.2032">
-</via>
-<wire x1="16.895" y1="8.5" x2="16.895" y2="7" width="0.254" layer="1"/>
-<wire x1="15" y1="8.5" x2="16.895" y2="8.5" width="0.254" layer="1"/>
 <wire x1="6.402" y1="9.271" x2="6.381" y2="9.25" width="0.254" layer="1"/>
 <wire x1="0.25" y1="13.381" x2="0.273" y2="13.358" width="0.254" layer="1"/>
@@
 <wire x1="-6.895" y1="0.4335875" x2="-6.895" y2="2" width="0.254" layer="1"/>
 <wire x1="-7.91429375" y1="-0.58570625" x2="-6.895" y2="0.4335875" width="0.254" layer="1"/>
-<contactref element="J1" pad="2"/>
 <wire x1="4.105" y1="-2.5" x2="2.9406" y2="-2.5" width="0.254" layer="1"/>
-<wire x1="25.46" y1="-2.54" x2="24.96" y2="-2.04" width="0.254" layer="1"/>
-<wire x1="24.96" y1="-2.04" x2="23.1165" y2="-2.0472875" width="0.254" layer="1"/>
 <via x="2.9406" y="-2.5" extent="1-16" drill="0.35">
-</via>
-<via x="23.1165" y="-2.0472875" extent="1-16" drill="0.35">
 </via>
 <via x="-0.508" y="-1.605" extent="1-16" drill="0.2032">
@@
 <wire x1="-9" y1="-3.5" x2="-8" y2="-4.5" width="0.254" layer="1"/>
 <wire x1="-8" y1="-4.5" x2="-7.81" y2="-4.65" width="0.254" layer="1"/>
-<wire x1="22.75" y1="-4.25" x2="23.5" y2="-4.25" width="0.254" layer="16"/>
-<wire x1="21.25" y1="-5.75" x2="22.75" y2="-4.25" width="0.254" layer="16"/>
-<wire x1="20.5" y1="-5.75" x2="21.25" y2="-5.75" width="0.254" layer="16"/>
-<wire x1="19.75" y1="-6.5" x2="20.5" y2="-5.75" width="0.254" layer="16"/>
-<wire x1="19.75" y1="-8.75" x2="19.75" y2="-6.5" width="0.254" layer="16"/>
-<wire x1="19.5" y1="-9" x2="19.75" y2="-8.75" width="0.254" layer="1"/>
-<wire x1="19.5" y1="-10" x2="19.5" y2="-9" width="0.254" layer="1"/>
-<wire x1="19.5" y1="-10" x2="19.5" y2="-10.5" width="0.254" layer="16"/>
 <wire x1="-1.5" y1="-9.25" x2="-1.5" y2="-12.5" width="0.254" layer="16"/>
 <wire x1="0.75" y1="-7" x2="-1.5" y2="-9.25" width="0.254" layer="16"/>
@@
 <via x="-9" y="-3.5" extent="1-16" drill="0.2032">
 </via>
-<via x="19.75" y="-8.75" extent="1-16" drill="0.2032">
-</via>
-<via x="19.5" y="-10" extent="1-16" drill="0.2032">
-</via>
 <via x="-1.5" y="-12.5" extent="1-16" drill="0.2032">
 </via>
@@
 </via>
 <wire x1="13.5" y1="-16.5" x2="10.80629375" y2="-13.80629375" width="0.254" layer="1"/>
-<wire x1="10.945875" y1="-13.6667125" x2="10.80629375" y2="-13.80629375" width="0.254" layer="16"/>
-<wire x1="19.5" y1="-10.5" x2="16.3332875" y2="-13.6667125" width="0.254" layer="16"/>
-<wire x1="16.3332875" y1="-13.6667125" x2="10.945875" y2="-13.6667125" width="0.254" layer="16"/>
 <via x="2.286" y="-0.663" extent="1-16" drill="0.2032">
 </via>
@@
 <wire x1="2.286" y1="-0.663" x2="2.199" y2="-0.75" width="0.254" layer="1"/>
 <wire x1="2.199" y1="-0.75" x2="1.75" y2="-0.75" width="0.254" layer="1"/>
-<wire x1="23.5" y1="-4.25" x2="23.5" y2="-2.4307875" width="0.254" layer="16"/>
-<wire x1="23.5" y1="-2.4307875" x2="23.1165" y2="-2.0472875" width="0.254" layer="16"/>
 </signal>
 <signal name="SCK">
