File: hardware/quadcopter.brd (EAGLE design)
At the start: 126.2 x 126.2 mm, 85 parts, among them J1 AVR_SPI_PRG_6-SMD, J2 HEADER-4POS-0.1IN-FEMALE-SMD-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, J3 HEADER-10POSTH-254X10, J4 HEADER-4POS-0.1IN-FEMALE-SMD-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, M1 MOTOR_PADS_GND-MOLEX-SMD, M2 MOTOR_PADS_GND-MOLEX-SMD, M3 MOTOR_PADS_GND-MOLEX-SMD, M4 MOTOR_PADS_GND-MOLEX-SMD, Q1 MOSFET-SI2302CDS-T1-E3CT-ND, Q2 MOSFET-SI2302CDS-T1-E3CT-ND, Q3 MOSFET-SI2302CDS-T1-E3CT-ND, Q4 MOSFET-SI2302CDS-T1-E3CT-ND, Q5 MOSFET-SI2302CDS-T1-E3CT-ND, Q6 MOSFET-SI2302CDS-T1-E3CT-ND, Q7 MOSFET-SI2302CDS-T1-E3CT-ND, Q8 MOSFET-SI2302CDS-T1-E3CT-ND, Q9 MOSFET-SI2302CDS-T1-E3CT-ND, SW1 PUSHBUTTON_SMD-VERTICAL-1, U1 ATMEGA128RFA1, U2 LSM-IMU-497-18367-1-NDIMU, Y1 CRYSTAL5X3

Commit message: FIXED THE CAPACITORS JESUS CHRIST
Parts:
- moved C2 25.4 mm to (-7.50, 11.5)
- moved C6 6.50 mm to (-7.50, 6.50)
Routing:
- net 3V: track 101.2 -> 85.4 mm
- net GND: track 51.2 -> 49.1 mm
- net PB5: track 60.8 -> 61.0 mm, vias 2 -> 3
